File: keeb.kicad_pcb (KiCad board)
At the start: 2 copper layers, 61 parts, among them J1 AVR-ISP-6, SW1 SW_Push, U1 ATmega32U4-AU, U2 PRTR5V0U2X, Y1 16MHz

Commit message: sex
Parts:
- moved C2 141.8 mm to (68.3, 88.1), turned to 270 degrees
- moved C8 140.6 mm to (69.1, 83.6), turned to 90 degrees
- moved C5 130.6 mm to (71.2, 87.3), turned to 0 degrees
- moved C1 5.56 mm to (66.7, 83.9)
- moved C4 5.56 mm to (46.3, 88.1)
- moved C6 5.56 mm to (63.5, 84.4)
- moved R1 5.56 mm to (66.9, 104.0)
- moved U1 5.56 mm to (59.5, 96.0)
- moved USB1 5.56 mm to (38.9, 79.4)
- moved Y1 5.56 mm to (58.9, 84.5)
- moved C3 5.56 mm to (53.2, 108.0)
- moved C7 5.56 mm to (54.0, 84.4)
- moved F1 5.56 mm to (46.0, 92.9)
- moved J1 5.56 mm to (44.5, 104.8)
- moved R2 5.56 mm to (35.7, 97.4)
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Connections:
- U1 pad 25: Net-(U1-Pad25) -> ROW0
- U1 pad 26: Net-(U1-Pad26) -> ROW1
- U1 pad 27: Net-(U1-Pad27) -> ROW2
- U1 pad 28: Net-(U1-Pad28) -> ROW3
- U1 pad 29: Net-(U1-Pad29) -> COL0
- U1 pad 30: Net-(U1-Pad30) -> COL1
- U1 pad 31: Net-(U1-Pad31) -> COL2
- U1 pad 32: Net-(U1-Pad32) -> COL3
- U1 pad 36: Net-(U1-Pad36) -> COL4
Routing:
- net COL4: track 0.00 -> 175.3 mm, vias 0 -> 10
- net ROW3: track 0.00 -> 160.1 mm
- net COL3: track 0.00 -> 153.8 mm, vias 0 -> 10
- net ROW2: track 0.00 -> 140.9 mm
- net ROW1: track 0.00 -> 124.0 mm
- net COL2: track 0.00 -> 122.2 mm, vias 0 -> 8
- net ROW0: track 0.00 -> 108.8 mm
- net COL1: track 0.00 -> 101.7 mm, vias 0 -> 8
- net COL0: track 0.00 -> 77.7 mm, vias 0 -> 7
- net +5V: track 60.5 -> 109.1 mm, vias 4 -> 9
- net GND: track 150.2 -> 174.2 mm
- net XTAL2: track 11.1 -> 23.7 mm, vias 2 -> 4
- net Net-(D4-Pad2): track 0.00 -> 5.97 mm
- net Net-(D19-Pad2): track 0.00 -> 5.97 mm
- net Net-(D2-Pad2): track 0.00 -> 5.97 mm
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