File: keeb.sch (KiCad schematic (older format))
At the start: 21 parts, among them J1 AVR-ISP-6, SW1 SW_Push, U1 ATmega32U4-AU, U2 PRTR5V0U2X, Y1 16MHz

Commit message: sex
Connections:
- net ROW0: now reaches U1.25 (PD4)
- net ROW1: now reaches U1.26 (PD6)
- net ROW2: now reaches U1.27 (PD7)
- net ROW3: now reaches U1.28 (PB4)
- net COL0: now reaches U1.29 (PB5)
- net COL1: now reaches U1.30 (PB6)
- net COL2: now reaches U1.31 (PC6)
- net COL3: now reaches U1.32 (PC7)
- net COL4: now reaches U1.36 (PF7)
- no-connect marks 3 -> 16
Changed lines of the file:
@@
 EESchema Schematic File Version 4
+LIBS:keeb-cache
 EELAYER 30 0
 EELAYER END
@@
 Wire Wire Line
 	1500 6650 1400 6650
+Text GLabel 2650 2950 2    50   Input ~ 0
+ROW0
+Text GLabel 2650 3150 2    50   Input ~ 0
+ROW1
+Text GLabel 2650 3250 2    50   Input ~ 0
+ROW2
+Text GLabel 2650 1750 2    50   Input ~ 0
+ROW3
+Text GLabel 2650 1850 2    50   Input ~ 0
+COL0
+Text GLabel 2650 1950 2    50   Input ~ 0
+COL1
+Text GLabel 2650 2250 2    50   Input ~ 0
+COL2
+Text GLabel 2650 2350 2    50   Input ~ 0
+COL3
+Text GLabel 2650 4250 2    50   Input ~ 0
+COL4
+NoConn ~ 2650 2050
+NoConn ~ 2650 2550
+NoConn ~ 2650 2650
+NoConn ~ 2650 2750
+NoConn ~ 2650 2850
+NoConn ~ 2650 3050
+NoConn ~ 2650 3550
+NoConn ~ 2650 3750
+NoConn ~ 2650 3850
+NoConn ~ 2650 3950
+NoConn ~ 2650 4050
+NoConn ~ 2650 4150
+NoConn ~ 2650 1350
 $EndSCHEMATC
